File: Hardware/CP_inverter.kicad_pcb (KiCad board)
At the start: 2 copper layers, 152 parts, among them J1 Weidmueller 1988610000, J2 Power in, J3 Weidmueller 2453690000, Q1 IRLML0030TRPBF, Q2 C3M0060065D, Q3 C3M0060065D, U1 LTV-217-C, U2 LTV-217-C, U3 LTV-217-C, U4 ICE3PCS01G, U5 T9VV1K15-12S, U6 L7815ACD2T, U7 B2424-1WR2, U8 UCC5390SCD

Commit message: new: Work in progress
Parts:
- added J2: PGood, Connector_Molex:Molex_SPOX_5268-02A_1x02_P2.50mm_Horizontal, F.Cu at (129.8, 229.6)
- added J3: PGood, Connector_Molex:Molex_SPOX_5268-02A_1x02_P2.50mm_Horizontal, F.Cu at (140.6, 229.6)
- added J4: PGood, Connector_Molex:Molex_SPOX_5268-02A_1x02_P2.50mm_Horizontal, F.Cu at (118.8, 229.6)
- R4: footprint Resistor_SMD:R_0805_2012Metric -> Resistor_SMD:R_1206_3216Metric
- moved D20 479.7 mm to (114.0, 231.0), turned to 90 degrees
- moved C10 459.1 mm to (121.8, 214.6), turned to 270 degrees
- moved C13 457.7 mm to (131.3, 225.1), turned to 270 degrees
- moved D14 454.5 mm to (103.3, 221.0)
- moved C30 450.5 mm to (109.8, 231.5), turned to 180 degrees
- moved R11 446.9 mm to (125.8, 214.6), turned to 90 degrees
- moved C16 440.3 mm to (127.6, 204.8), turned to 90 degrees
- moved C39 439.6 mm to (110.5, 212.8), turned to 90 degrees
- moved C18 429.3 mm to (149.3, 199.8)
- moved R12 427.9 mm to (123.8, 214.6), turned to 90 degrees
- moved R9 427.4 mm to (136.6, 201.3), turned to 90 degrees
- moved D5 412.5 mm to (118.3, 224.8), turned to 270 degrees
- moved R16 407.4 mm to (133.8, 225.1), turned to 90 degrees
- moved D6 405.8 mm to (129.3, 224.8), turned to 270 degrees
- moved C23 404.8 mm to (88.5, 216.5), turned to 90 degrees
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- renumbered J2 to J5, J3 to J6
Connections:
- net CS2 renamed GND
Routing:
- net GATE: track 0.00 -> 68.1 mm
- net Net-(C23-Pad1): track 0.00 -> 63.8 mm
- net +15V: track 0.00 -> 53.0 mm
- net Net-(C8-Pad1): track 0.00 -> 51.8 mm
- net -5V: track 0.00 -> 38.9 mm
- net Net-(C5-Pad1): track 0.00 -> 34.0 mm
- net GND: track 0.00 -> 31.9 mm, vias 0 -> 131
- net VBUS: track 0.00 -> 30.9 mm
- net Net-(C18-Pad1): track 0.00 -> 26.8 mm
- net Net-(C21-Pad1): track 0.00 -> 26.4 mm
- net Earth: track 0.00 -> 25.8 mm
- net Net-(C4-Pad1): track 0.00 -> 25.8 mm
- net Net-(C1-Pad1): track 0.00 -> 25.1 mm
- net (no net): track 0.00 -> 24.6 mm
- net VCC: track 0.00 -> 20.5 mm, vias 0 -> 11
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- added copper zone on F.Cu, net VBUS
- added copper zone on F.Cu, net VCC

Commit message: new: Work in progress, filter layout
Parts:
- moved R15 90.0 mm to (390.2, 215.5)
- moved R14 89.1 mm to (390.2, 220.6)
- moved R13 88.5 mm to (390.2, 226.0)
- moved F1 40.4 mm to (353.0, 225.0), turned to 180 degrees
- moved R34 14.5 mm to (163.0, 173.0), turned to 180 degrees
- moved C55 11.0 mm to (385.5, 193.0)
- moved C20 10.5 mm to (204.0, 189.0)
- moved D9 10.5 mm to (204.0, 192.0)
- moved R33 8.94 mm to (181.5, 97.0), turned to 0 degrees
- moved C14 8.19 mm to (269.5, 211.5)
- moved R35 8.06 mm to (174.0, 97.0), turned to 180 degrees
- moved R36 7.28 mm to (170.0, 166.0), turned to 0 degrees
- moved C15 7.17 mm to (269.5, 201.5)
- moved R25 7.16 mm to (194.5, 231.5)
- moved C19 5.27 mm to (218.5, 218.0)
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Connections:
- Q2 pad 2: GND -> Net-(D16-Pad2)
- Q2 pad 3: Net-(D16-Pad2) -> GND
- Q3 pad 2: GND -> Net-(D18-Pad2)
- Q3 pad 3: Net-(D18-Pad2) -> GND
Routing:
- net VBUS: track 30.9 -> 110.7 mm
- net Net-(C7-Pad2): track 15.5 -> 0.00 mm
- net Net-(C6-Pad1): track 14.9 -> 0.00 mm
- net GATE: track 68.1 -> 79.1 mm
- net Net-(Q2-Pad1): track 0.00 -> 10.6 mm
- net Net-(C20-Pad2): track 10.2 -> 0.00 mm
- net Net-(Q3-Pad1): track 0.00 -> 10.1 mm
- net Net-(C20-Pad1): track 9.76 -> 0.00 mm
- net Earth: track 25.8 -> 21.1 mm
- net Net-(R44-Pad2): track 0.00 -> 2.61 mm
- net Net-(R43-Pad2): track 0.00 -> 2.54 mm
- net GND: vias 131 -> 139
- added copper zone on F.Cu, net Earth
- added copper zone on F.Cu, net GND
- added copper zone on F.Cu, net Net-(C6-Pad1)
- added copper zone on F.Cu, net Net-(C7-Pad2)
- added copper zone on F.Cu, net Net-(D16-Pad2)
- added copper zone on F.Cu, net Net-(D18-Pad2)
- added copper zone on F.Cu, net Net-(F1-Pad1)
Other:
- net class HV added: clearance 2.5, trace_width 0.25, via_dia 0.8, via_drill 0.4

Commit message: new: first rev
Parts:
- R31, R32: moved to B.Cu
- moved R31 56.1 mm to (73.5, 183.4)
- moved R32 47.3 mm to (73.5, 179.2)
- moved C22 23.7 mm to (38.2, 158.4), turned to 270 degrees
- moved R25 22.1 mm to (175.5, 220.2)
- moved D2 20.6 mm to (152.5, 233.8)
- moved D3 20.0 mm to (152.5, 227.0), turned to 180 degrees
- moved C1 19.9 mm to (125.1, 221.6)
- moved C10 19.9 mm to (102.8, 220.6)
- moved C11 19.9 mm to (108.8, 220.6)
- moved C12 19.9 mm to (126.3, 207.3)
- moved C13 19.9 mm to (112.3, 231.1)
- moved C16 19.9 mm to (108.6, 210.8)
- moved C18 19.9 mm to (130.3, 205.8)
- moved C2 19.9 mm to (123.1, 231.1)
- moved C21 19.9 mm to (130.4, 223.1)
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Routing:
- net Earth: track 21.1 -> 510.5 mm, vias 0 -> 12
- net VCC: track 20.5 -> 378.7 mm, vias 11 -> 20
- net -5V: track 38.9 -> 224.5 mm, vias 0 -> 3
- net Net-(C27-Pad1): track 0.00 -> 179.7 mm
- net Net-(C28-Pad1): track 0.00 -> 169.6 mm
- net +15V: track 53.0 -> 212.9 mm, vias 0 -> 3
- net GND: track 31.9 -> 188.0 mm, vias 139 -> 140
- net AC_IN2: track 0.00 -> 145.5 mm, vias 0 -> 48
- net Net-(C50-Pad1): track 5.47 -> 135.4 mm, vias 0 -> 6
- net VBUS: track 110.7 -> 217.7 mm
- net VB_OK: track 11.5 -> 90.5 mm, vias 0 -> 3
- net AC_IN1: track 0.00 -> 78.0 mm
- net Net-(C6-Pad1): track 0.00 -> 64.6 mm
- net CS1: track 0.00 -> 64.0 mm, vias 0 -> 33
- net Net-(C20-Pad2): track 0.00 -> 40.1 mm
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- added copper zone on F.Cu, net AC_IN1
- added copper zone on B.Cu, net AC_IN2
- added copper zone on F.Cu, net AC_IN2
- added copper zone on In2.Cu, net AC_IN2
- added copper zone on B.Cu, net CS1
- added copper zone on F.Cu, net CS1
- added copper zone on B.Cu, net GND
- added copper zone on In1.Cu, net GND
- added copper zone on F.Cu, net Net-(C14-Pad1)
- added copper zone on F.Cu, net Net-(C15-Pad2)
- added copper zone on F.Cu, net Net-(C27-Pad1)
- added copper zone on F.Cu, net Net-(C28-Pad1)
- added copper zone on B.Cu, net Net-(D11-Pad2)
- added copper zone on F.Cu, net Net-(D11-Pad2)
- added copper zone on In2.Cu, net Net-(D11-Pad2)
- added copper zone on B.Cu, net VCC
- added copper zone on In2.Cu, net VCC
Other:
- board outline added: 380 x 200 mm
- copper layers 2 -> 4

Commit message: new: rev. 1.0. fixes
Parts:
- added H1: MountingHole, MountingHole:MountingHole_3.2mm_M3_DIN965, F.Cu at (26.0, 246.0)
- added H2: MountingHole, MountingHole:MountingHole_3.2mm_M3_DIN965, F.Cu at (26.0, 56.0)
- added H3: MountingHole, MountingHole:MountingHole_3.2mm_M3_DIN965, F.Cu at (396.0, 56.0)
- added H4: MountingHole, MountingHole:MountingHole_3.2mm_M3_DIN965, F.Cu at (396.0, 246.0)
- added H5: MountingHole, MountingHole:MountingHole_3.2mm_M3_DIN965, F.Cu at (205.0, 56.0)
- added H6: MountingHole, MountingHole:MountingHole_3.2mm_M3_DIN965, F.Cu at (205.0, 131.0)
- added H7: MountingHole, MountingHole:MountingHole_3.2mm_M3_DIN965, F.Cu at (205.0, 246.0)
- added R31: DNP, Resistor_SMD:R_2512_6332Metric, B.Cu at (73.5, 179.0)
- added R32: DNP, Resistor_SMD:R_2512_6332Metric, B.Cu at (73.5, 175.0)
- moved R34 3.75 mm to (73.5, 183.0)
- moved R33 3.59 mm to (73.5, 187.0)
- moved L2 1.00 mm to (129.0, 126.0)
- moved L3 1.00 mm to (129.0, 128.0)
- moved R40 0.75 mm to (63.5, 208.5)
- moved F1 0.50 mm to (353.0, 222.5)
- moved D2 0.25 mm to (152.5, 233.5)
- moved F2 0.10 mm to (81.5, 237.8)
- renumbered R31 to R33, R32 to R34, R33 to R35, R34 to R36, R35 to R37, R36 to R38, R37 to R39, R38 to R40, R39 to R41, R40 to R42, R41 to R43, R42 to R44, R43 to R45, R44 to R46, R45 to R47
Routing:
- net Earth: track 510.5 -> 310.3 mm
- net AC_IN1: track 78.0 -> 33.7 mm
- net GND: track 188.0 -> 210.4 mm, vias 140 -> 308
- net Net-(D11-Pad2): track 9.89 -> 0.00 mm, vias 80 -> 121
- net CS1: track 64.0 -> 70.2 mm, vias 33 -> 65
- net AC_IN2: track 145.5 -> 149.4 mm, vias 48 -> 101
- net Net-(C31-Pad1): track 19.5 -> 22.6 mm
- net Net-(R13-Pad1): track 0.00 -> 2.53 mm
- net Net-(C27-Pad1): track 179.7 -> 182.1 mm
- net Net-(R14-Pad1): track 0.00 -> 2.12 mm
- net Net-(C6-Pad1): track 64.6 -> 63.3 mm
- net VBUS: track 217.7 -> 216.6 mm
- net Net-(C4-Pad1): track 25.8 -> 24.9 mm
- net Net-(D21-Pad2): track 1.40 -> 2.15 mm
- net VCC: track 378.7 -> 378.2 mm
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Other:
- board text added: "400VDC out"
- board text added: "85-265VAC in"
- board text added: "Caution! High voltage."
- board text added: "Earth"
- board text added: "GND"
- board text added: "L"
- board text added: "N"
- board text added: "PFC module"
- board text added: "VOUT"
- board text added: "ver. 1.0"

Commit message: new: production files added
Parts:
- moved C37 13.0 mm to (245.2, 92.8)
- moved C38 13.0 mm to (285.2, 92.8)
- moved C41 13.0 mm to (325.2, 92.8)
- moved C52 13.0 mm to (245.2, 97.8)
- moved C53 13.0 mm to (285.2, 97.8)
- moved C54 13.0 mm to (325.2, 97.8)
- moved J6 7.07 mm to (371.2, 130.8)
Routing:
- net VBUS: track 216.6 -> 225.8 mm
- net GND: track 210.4 -> 201.6 mm, vias 308 -> 366
- net AC_IN2: track 149.4 -> 148.2 mm
- net BOFO_ENBL-: track 13.7 -> 12.8 mm
- net Earth: vias 12 -> 0
Other:
- board text added: "400VDC"
- board text added: "85-265VAC"
